File: HeartPendant/Pendant.kicad_sch (KiCad schematic)
At the start: 56 parts, among them J4 Bat +, J5 Bat -, J6 USB_C_Receptacle_USB2.0_16P, Q1 AO3401A, Q2 2N7002, SW3 SW_Boot, SW4 SW_SPDT, U6 MCP73831-2-OT, U7 ESP32-C3-MINI-1-N4X, U8 AP2112K-3.3, U9 USBLC6-2SC6

Commit message: Added: Started on PCB, made custom outline, finished routing Bracelet
Parts:
- removed J4: Bat +, Package_TO_SOT_SMD:SOT-23-5, symbol Connector:Conn_01x01_Pin
- removed J5: Bat -, Package_TO_SOT_SMD:SOT-23-5, symbol Connector:Conn_01x01_Pin
- added J3: Bat, Connector_PinHeader_2.54mm:PinHeader_1x02_P2.54mm_Vertical, symbol Connector:Conn_01x02_Pin
- C10: footprint (none) -> Capacitor_SMD:C_0805_2012Metric
- C11, C12, C14: footprint Package_TO_SOT_SMD:SOT-23-5 -> Capacitor_SMD:C_0603_1608Metric
- C13, C9: footprint (none) -> Capacitor_SMD:C_0603_1608Metric
- C15: renamed from C17; footprint Package_TO_SOT_SMD:SOT-23 -> Capacitor_SMD:C_0603_1608Metric
- C16: renamed from C20; footprint Package_TO_SOT_SMD:SOT-23 -> Capacitor_SMD:C_0603_1608Metric
- C17: renamed from C23; footprint Package_TO_SOT_SMD:SOT-23 -> Capacitor_SMD:C_0603_1608Metric
- C18, C22: footprint Package_TO_SOT_SMD:SOT-23 -> Capacitor_SMD:C_0603_1608Metric
- C19: renamed from C21; footprint Package_TO_SOT_SMD:SOT-23 -> Capacitor_SMD:C_0603_1608Metric
- C20: renamed from C24; footprint Package_TO_SOT_SMD:SOT-23 -> Capacitor_SMD:C_0603_1608Metric
- C21: renamed from C19; footprint Package_TO_SOT_SMD:SOT-23 -> Capacitor_SMD:C_0603_1608Metric
- C23: renamed from C25; footprint Package_TO_SOT_SMD:SOT-23 -> Capacitor_SMD:C_0603_1608Metric
- C24: renamed from C15; footprint Package_TO_SOT_SMD:SOT-23-5 -> Capacitor_SMD:C_0603_1608Metric
- C25: renamed from C28; footprint Package_TO_SOT_SMD:SOT-23 -> Capacitor_SMD:C_0603_1608Metric
- C26: renamed from C27; footprint Package_TO_SOT_SMD:SOT-23 -> Capacitor_SMD:C_0603_1608Metric
- C27: renamed from C26; footprint Package_TO_SOT_SMD:SOT-23 -> Capacitor_SMD:C_0603_1608Metric
- C28: renamed from C16; footprint Package_TO_SOT_SMD:SOT-23-5 -> Capacitor_SMD:C_0603_1608Metric
- D2: footprint LED_SMD:LED_Cree-XHP50_3V_HighDensity -> LED_SMD:LED_0603_1608Metric
- J4: renamed from J6; footprint Package_DFN_QFN:WDFN-10-1EP_3x3mm_P0.5mm_EP1.8x2.5mm -> Connector_USB:USB_C_Receptacle_HRO_TYPE-C-31-M-12
- R10, R11, R13, R16: footprint (none) -> Resistor_SMD:R_0603_1608Metric
- R12, R14, R15: footprint RF_Module:ESP32-C3-DevKitM-1 -> Resistor_SMD:R_0603_1608Metric
- R17: renamed from R20; footprint Package_TO_SOT_SMD:SOT-23 -> Resistor_SMD:R_0603_1608Metric
- R18: renamed from R19; footprint Package_TO_SOT_SMD:SOT-23 -> Resistor_SMD:R_0603_1608Metric
- R19: renamed from R21; footprint Package_TO_SOT_SMD:SOT-23 -> Resistor_SMD:R_0603_1608Metric
- R20: renamed from R17; footprint (none) -> Resistor_SMD:R_0603_1608Metric
- R21: renamed from R18; footprint (none) -> Resistor_SMD:R_0603_1608Metric
- SW3: footprint Package_DIP:DIP-24_W7.62mm -> HX_Push_SW:SW-SMD_4P-L4.2-W3.4-P2.15-LS5.2
- SW4: footprint Button_Switch_THT:SW_Slide-03_Wuerth-WS-SLTV_10x2.5x6.4_P2.54mm -> MSK12C02:SW-TH_MSK12C02
- renumbered D8 to D10, D14 to D12, D12 to D14, D6 to D4, D9 to D5, D4 to D6, D10 to D8, D5 to D9, Q2 to Q1, Q1 to Q2, U9 to U8, U8 to U9
Connections:
- net GND_P: now also J3.1 (Pin_1)
- net VBAT: now also J3.2 (Pin_2)

Commit message: Finished pendant routing, added production files
Parts:
- C10: LCSC Part (none) -> C1713
- C11, C12, C14: LCSC Part (none) -> C1705
- C13, C15, C16, C17, C18, C19, C20, C21, C22, C23, C25, C26, C27: LCSC Part (none) -> C1590
- C24, C28, C9: LCSC Part (none) -> C1592
- D10, D11, D12, D13, D14, D3, D4, D5, D6, D7, D8, D9: LCSC Part (none) -> C5149201
- D2: LCSC Part (none) -> C2286
- J3: now not fitted; now left out of the parts list
- J4: LCSC Part (none) -> C165948
- Q1: LCSC Part (none) -> C8545
- Q2: LCSC Part (none) -> C478608
- R10, R11, R18: LCSC Part (none) -> C14675
- R12, R13, R14, R15, R17: LCSC Part (none) -> C15401
- R16: LCSC Part (none) -> C23179
- R19: LCSC Part (none) -> C22104
- R20, R21: LCSC Part (none) -> C14677
- SW3: LCSC Part (none) -> C55200589
- SW4: LCSC Part (none) -> C431540
- U6: LCSC Part (none) -> C14879
- U8: LCSC Part (none) -> C7519
- U9: LCSC Part (none) -> C51118
